Commit message: project done

File: ros-ws/src/robotteknik/robot_models/franka_description/robots/panda_arm_old.xacro (robot description, xacro)
@@ -18,4 +18,9 @@
         </geometry>
       </visual>
+      <collision>
+        <geometry>
+          <mesh filename="package://${description_pkg}/meshes/collision/link0.stl"/>
+        </geometry>
+      </collision>
       <!-- for simulation -->
       <inertial>
@@ -32,4 +37,9 @@
         </geometry>
       </visual>
+      <collision>
+        <geometry>
+          <mesh filename="package://${description_pkg}/meshes/collision/link1.stl"/>
+        </geometry>
+      </collision>
       <!-- for simulation -->
       <inertial>
@@ -57,4 +67,9 @@
         </geometry>
       </visual>
+      <collision>
+        <geometry>
+          <mesh filename="package://${description_pkg}/meshes/collision/link2.stl"/>
+        </geometry>
+      </collision>
       <!-- for simulation -->
       <inertial>
@@ -82,4 +97,9 @@
         </geometry>
       </visual>
+      <collision>
+        <geometry>
+          <mesh filename="package://${description_pkg}/meshes/collision/link3.stl"/>
+        </geometry>
+      </collision>
       <!-- for simulation -->
       <inertial>
@@ -107,4 +127,9 @@
         </geometry>
       </visual>
+      <collision>
+        <geometry>
+          <mesh filename="package://${description_pkg}/meshes/collision/link4.stl"/>
+        </geometry>
+      </collision>
       <!-- for simulation -->
       <inertial>
@@ -132,4 +157,9 @@
         </geometry>
       </visual>
+      <collision>
+        <geometry>
+          <mesh filename="package://${description_pkg}/meshes/collision/link5.stl"/>
+        </geometry>
+      </collision>
       <!-- for simulation -->
       <inertial>
@@ -157,4 +187,9 @@
         </geometry>
       </visual>
+      <collision>
+        <geometry>
+          <mesh filename="package://${description_pkg}/meshes/collision/link6.stl"/>
+        </geometry>
+      </collision>
       <!-- for simulation -->
       <inertial>
@@ -182,4 +217,9 @@
         </geometry>
       </visual>
+      <collision>
+        <geometry>
+          <mesh filename="package://${description_pkg}/meshes/collision/link7.stl"/>
+        </geometry>
+      </collision>
       <!-- for simulation -->
       <inertial>
